File: Hardware/I2C_Breakout_Block.brd (EAGLE design)
At the start: 30.5 x 44.5 mm, 25 parts, among them U2 PCA9306

Commit message: Ready for reds Tweak schematic, add value to regulator No known to-do items
Parts:
- U1: value (none) -> MIC5205
Changed lines of the file:
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@@
 <setting verticaltext="up"/>
 </settings>
-<grid distance="0.001" unitdist="inch" unit="inch" style="lines" multiple="1" display="yes" altdistance="0.005" altunitdist="inch" altunit="inch"/>
+<grid distance="0.05" unitdist="inch" unit="inch" style="lines" multiple="1" display="yes" altdistance="0.005" altunitdist="inch" altunit="inch"/>
 <layers>
 <layer number="1" name="Top" color="4" fill="1" visible="yes" active="yes"/>
-<layer number="2" name="Route2" color="1" fill="3" visible="yes" active="yes"/>
+<layer number="2" name="Route2" color="1" fill="3" visible="no" active="yes"/>
 <layer number="15" name="Route15" color="4" fill="6" visible="no" active="yes"/>
 <layer number="16" name="Bottom" color="1" fill="1" visible="yes" active="yes"/>
@@
 <layer number="20" name="Dimension" color="15" fill="1" visible="yes" active="yes"/>
 <layer number="21" name="tPlace" color="16" fill="1" visible="yes" active="yes"/>
-<layer number="22" name="bPlace" color="14" fill="1" visible="no" active="yes"/>
+<layer number="22" name="bPlace" color="14" fill="1" visible="yes" active="yes"/>
 <layer number="23" name="tOrigins" color="15" fill="1" visible="yes" active="yes"/>
-<layer number="24" name="bOrigins" color="15" fill="1" visible="no" active="yes"/>
+<layer number="24" name="bOrigins" color="15" fill="1" visible="yes" active="yes"/>
 <layer number="25" name="tNames" color="7" fill="1" visible="no" active="yes"/>
 <layer number="26" name="bNames" color="7" fill="1" visible="no" active="yes"/>
@@
 <layer number="43" name="vRestrict" color="2" fill="10" visible="no" active="yes"/>
 <layer number="44" name="Drills" color="7" fill="1" visible="no" active="yes"/>
-<layer number="45" name="Holes" color="7" fill="1" visible="no" active="yes"/>
+<layer number="45" name="Holes" color="7" fill="1" visible="yes" active="yes"/>
 <layer number="46" name="Milling" color="3" fill="1" visible="no" active="yes"/>
-<layer number="51" name="tDocu" color="6" fill="1" visible="no" active="yes"/>
+<layer number="51" name="tDocu" color="6" fill="1" visible="yes" active="yes"/>
 <layer number="3" name="Route3" color="4" fill="3" visible="no" active="no"/>
 <layer number="4" name="Route4" color="1" fill="4" visible="no" active="no"/>
@@
 <text x="19.05" y="43.18" size="1.6764" layer="21" font="vector" ratio="15" rot="R270" align="center-left">SCL</text>
 <text x="31.75" y="-2.54" size="1.778" layer="51">Note: Units are in Inches</text>
+<wire x1="17.018" y1="27.94" x2="17.399" y2="27.94" width="0.1524" layer="41"/>
 </plain>
 <attributes>
@@
 <element name="JP2" library="SparkFun-Connectors" package="1X04_SMD_RA_FEMALE" value="" x="15.24" y="40.132" rot="R180"/>
 <element name="SJ1" library="SparkFun-Passives" package="PAD-JUMPER-3-2OF3_NC_BY_TRACE_YES_SILK_FULL_BOX" value="Power Select" x="12.192" y="23.114" rot="R180"/>
-<element name="U1" library="SparkFun-PowerIC" package="SOT23-5" value="" x="12.192" y="19.558">
+<element name="U1" library="SparkFun-PowerIC" package="SOT23-5" value="MIC5205" x="12.192" y="19.558">
 <attribute name="PROD_ID" value="VREG-00822" x="12.192" y="19.558" size="1.778" layer="27" display="off"/>
 </element>
